File: Hardware/P1_Extender/P1_Extender.kicad_pcb (KiCad board)
At the start: 2 copper layers, 51 x 47 mm, 8 parts, among them J1 RJ12, U1 6N137, U2 WeMos_D1_mini, U3 6N137

Commit message: Added new hardware version to fix the issues
Parts:
- added JP2: Factory Reset, Connector_PinHeader_2.54mm:PinHeader_1x02_P2.54mm_Vertical, F.Cu at (144.5, 113.0)
Connections:
- U1 pad 3: GND -> Net-(U1-C)
- U2 pad 14: unconnected-(U2-SCL/D1-Pad14) -> Net-(U1-C)
- U2 pad 5: unconnected-(U2-MISO/D6-Pad5) -> Net-(JP2-A)
Routing:
- net Net-(JP2-A): track 0.00 -> 16.5 mm
- net GND: track 154.3 -> 157.3 mm
- net Net-(JP1-B): track 11.0 -> 11.9 mm
Other:
- board text added: "factory"
- board text added: "reset"
